File: rusb-pd-second/rusb-pd-second.kicad_sch (KiCad schematic)
At the start: 15 parts, among them J1 Conn_02x05_Counter_Clockwise, J2 Conn_01x02, U1 AMS1117-3.3, U3 FUSB302BMPX, U4 CH32V003FxUx

Commit message: lotta changes (described in the articel)
Parts:
- added C5, C6: 100n, Capacitor_SMD:C_0603_1608Metric, symbol Device:C_Small
- added D1: 3V6, Diode_SMD:D_0805_2012Metric, symbol Device:D_Zener_Small
- added D2: LED1, LED_SMD:LED_0603_1608Metric, symbol Device:LED_Small
- added D3: LED2, LED_SMD:LED_0603_1608Metric, symbol Device:LED_Small
- added J3: qwiic, Connector_JST:JST_SH_SM04B-SRSS-TB_1x04-1MP_P1.00mm_Horizontal, symbol Connector_Generic_MountingPin:Conn_01x04_MountingPin
- added Q1: AO3401, Package_TO_SOT_SMD:SOT-23, symbol Device:Q_PMOS_GSD
- added Q2: BC847, Package_TO_SOT_SMD:SOT-23, symbol Transistor_BJT:BC847
- added R10, R3, R8: 1K5, Resistor_SMD:R_0402_1005Metric, symbol Device:R_Small
- added R11, R12: 5.1K, Resistor_SMD:R_0402_1005Metric, symbol Device:R_Small
- added R4: 15K, Resistor_SMD:R_0402_1005Metric, symbol Device:R_Small
- added R9: 4K7, Resistor_SMD:R_0402_1005Metric, symbol Device:R_Small
- added SW1: SW_DIP_x03, rusb-pd-second:SW-SMD_6P-P1.27_EU-03KS, symbol Switch:SW_DIP_x03
- R1, R2: value 3K3 -> 1K5
Connections:
- net +3.3V: now also C5.1, C6.1, D3.2 (A), J3.2 (Pin_2), SW1.4
- net F_SCL: now also J3.4 (Pin_4)
- net F_SDA: now also J3.3 (Pin_3)
- net GND: now also U4.21 (VSS), C5.2, C6.2, D1.2 (A), D2.1 (K), J3.1 (Pin_1), J3.MP (MountPin), Q2.2 (E), R3.2, SW1.5, SW1.6; no longer U4.0 (VSS)
- net TYPEC_VBUS: now also U1.3 (VI), Q1.2 (S), R4.1, R8.2; no longer L1.1, R7.2
- net VBUS: no longer U1.3 (VI), U3.2 (VBUS)
- net VBUS_EN: now reaches U4.1 (PD7)
- net VBUS_EN: now also R10.1
- net VBUS_ADC: now reaches U4.11 (PC4)
- net VBUS_ADC: now also D1.1 (K), R3.1, R4.2
- net CFG3: now reaches U4.16 (PD2)
- net CFG3: now also SW1.3
- net CFG1: now reaches U4.2 (PA1)
- net CFG1: now also SW1.1
- net CFG2: now reaches U4.3 (PA2)
- net CFG2: now also SW1.2
- net LED: now reaches U4.7 (PC0)
- net LED: now also R11.2, R12.2
- new net: D3.1 (K), R12.1
- new net: D2.2 (A), R11.1
- new net: L1.1, Q1.3 (D), R7.2
- new net: Q2.1 (B), R10.2
- new net: Q1.1 (G), R8.1, R9.2
- new net: Q2.3 (C), R9.1
Other:
- moved on the sheet: C1, C3, C4, L1, R6, R7
